File: lm4862-board-1.kicad_sch (KiCad schematic)
At the start: 14 parts, among them J1 Conn_01x02, J2 Conn_01x06, J3 Conn_01x02

Commit message: Updated docs
Other:
- note added: "Power"
- note removed: "POWER"
- moved on the sheet: C1, H1, H2, H3, H4, J3
